File: hardware design/LEDs.kicad_sch (KiCad schematic)
At the start: 27 parts

Commit message: library name updating, footprint swaps
Parts:
- D10, D11, D12, D13, D14, D15, D16, D17, D18, D19, D20, D21, D22, D23, D24, D25, D3, D4, D5, D6, D7, D8, D9: footprint EURORACK:SK6812MINIE -> benjiaomodular:SK6812MINIE
Changed lines of the file:
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@@
 			)
 		)
-		(property "Footprint" "EURORACK:SK6812MINIE"
+		(property "Footprint" "benjiaomodular:SK6812MINIE"
 			(at 89.154 60.706 0)
 			(effects
@@
 			)
 		)
-		(property "Footprint" "EURORACK:SK6812MINIE"
+		(property "Footprint" "benjiaomodular:SK6812MINIE"
 			(at 133.35 103.632 0)
 			(effects
@@
 			)
 		)
-		(property "Footprint" "EURORACK:SK6812MINIE"
+		(property "Footprint" "benjiaomodular:SK6812MINIE"
 			(at 110.998 103.632 0)
 			(effects
@@
 			)
 		)
-		(property "Footprint" "EURORACK:SK6812MINIE"
+		(property "Footprint" "benjiaomodular:SK6812MINIE"
 			(at 201.168 147.574 0)
 			(effects
@@
 			)
 		)
-		(property "Footprint" "EURORACK:SK6812MINIE"
+		(property "Footprint" "benjiaomodular:SK6812MINIE"
 			(at 178.308 147.574 0)
 			(effects
@@
 			)
 		)
-		(property "Footprint" "EURORACK:SK6812MINIE"
+		(property "Footprint" "benjiaomodular:SK6812MINIE"
 			(at 179.324 60.706 0)
 			(effects
@@
 			)
 		)
-		(property "Footprint" "EURORACK:SK6812MINIE"
+		(property "Footprint" "benjiaomodular:SK6812MINIE"
 			(at 223.52 103.632 0)
 			(effects
@@
 			)
 		)
-		(property "Footprint" "EURORACK:SK6812MINIE"
+		(property "Footprint" "benjiaomodular:SK6812MINIE"
 			(at 133.35 147.574 0)
 			(effects
@@
 			)
 		)
-		(property "Footprint" "EURORACK:SK6812MINIE"
+		(property "Footprint" "benjiaomodular:SK6812MINIE"
 			(at 89.154 147.574 0)
 			(effects
@@
 			)
 		)
-		(property "Footprint" "EURORACK:SK6812MINIE"
+		(property "Footprint" "benjiaomodular:SK6812MINIE"
 			(at 201.168 103.632 0)
 			(effects
@@
 			)
 		)
-		(property "Footprint" "EURORACK:SK6812MINIE"
+		(property "Footprint" "benjiaomodular:SK6812MINIE"
 			(at 156.972 60.706 0)
 			(effects
@@
 			)
 		)
-		(property "Footprint" "EURORACK:SK6812MINIE"
+		(property "Footprint" "benjiaomodular:SK6812MINIE"
 			(at 178.562 103.632 0)
 			(effects
@@
 			)
 		)
-		(property "Footprint" "EURORACK:SK6812MINIE"
+		(property "Footprint" "benjiaomodular:SK6812MINIE"
 			(at 66.04 103.632 0)
 			(effects
@@
 			)
 		)
-		(property "Footprint" "EURORACK:SK6812MINIE"
+		(property "Footprint" "benjiaomodular:SK6812MINIE"
 			(at 88.392 103.632 0)
 			(effects
@@
 			)
 		)
-		(property "Footprint" "EURORACK:SK6812MINIE"
+		(property "Footprint" "benjiaomodular:SK6812MINIE"
 			(at 111.76 60.706 0)
 			(effects
@@
 			)
 		)
-		(property "Footprint" "EURORACK:SK6812MINIE"
+		(property "Footprint" "benjiaomodular:SK6812MINIE"
 			(at 134.112 60.706 0)
 			(effects
@@
 			)
 		)
-		(property "Footprint" "EURORACK:SK6812MINIE"
+		(property "Footprint" "benjiaomodular:SK6812MINIE"
 			(at 66.802 147.574 0)
 			(effects
@@
 			)
 		)
-		(property "Footprint" "EURORACK:SK6812MINIE"
+		(property "Footprint" "benjiaomodular:SK6812MINIE"
 			(at 201.93 60.706 0)
 			(effects
@@
 			)
 		)
-		(property "Footprint" "EURORACK:SK6812MINIE"
+		(property "Footprint" "benjiaomodular:SK6812MINIE"
 			(at 66.802 60.706 0)
 			(effects
@@
 			)
 		)
-		(property "Footprint" "EURORACK:SK6812MINIE"
+		(property "Footprint" "benjiaomodular:SK6812MINIE"
 			(at 111.76 147.574 0)
 			(effects
@@
 			)
 		)
-		(property "Footprint" "EURORACK:SK6812MINIE"
+		(property "Footprint" "benjiaomodular:SK6812MINIE"
 			(at 156.21 103.632 0)
 			(effects
@@
 			)
 		)
-		(property "Footprint" "EURORACK:SK6812MINIE"
+		(property "Footprint" "benjiaomodular:SK6812MINIE"
 			(at 155.702 147.574 0)
 			(effects
@@
 			)
 		)
-		(property "Footprint" "EURORACK:SK6812MINIE"
+		(property "Footprint" "benjiaomodular:SK6812MINIE"
 			(at 224.282 60.706 0)
 			(effects
