File: hardware design/dsug_cctv_BOARD.kicad_pcb (KiCad board)
At the start: 2 copper layers, 120 x 102.5 mm, 245 parts, among them J1 Conn_02x05_Top_Bottom, J10 JACK, J11 JACK, J12 JACK, J13 JACK, J14 JACK, J15 JACK, J16 JACK, J17 JACK, J18 JACK, J19 JACK, J2 JACK, J20 JACK, J3 TYPEC-304-ACP16, J4 JACK, J5 JACK, J6 JACK, J7 JACK, J8 JACK, J9 JACK, Q1 MMBT3904, Q2 MMBT3904, Q3 MMBT3904, Q4 MMBT3904, SW1 TS-1187A-B-A-B, SW3 SW_Push, SW4 SW_SPDT_MSM, SW5 SW_SPDT_MSM, U1 AMS1117-3.3, U10 MCP6004, U11 MCP6004, U12 TL074, U13 RP2040, U14 TL074, U2 W25Q128JVS, U3 AMS1117-5.0, U4 CD4051B, U5 TL074, U6 CD4051B, U7 MCP6004, U8 LM4040DIM3-10.0/NOPB, U9 TL074, Y1 Crystal_GND24

Commit message: pcb rev2.5
Parts:
- removed C3: 10uF, Capacitor_THT:CP_Radial_D5.0mm_P2.50mm
- removed Q1, Q2: MMBT3904, Package_TO_SOT_SMD:SOT-23
- removed R100, R47, R88, R99: 1k, Resistor_SMD:R_0603_1608Metric
- added C54: 100nF, Capacitor_SMD:C_0603_1608Metric, B.Cu at (98.1, 43.5)
- added C55: 10uF, Capacitor_THT:CP_Radial_D5.0mm_P2.50mm, F.Cu at (93.1, 46.7)
- added C56: 10uF, Capacitor_THT:CP_Radial_D5.0mm_P2.50mm, F.Cu at (190.3, 55.7)
- added C57: 10uF, Capacitor_THT:CP_Radial_D5.0mm_P2.50mm, F.Cu at (190.3, 46.9)
- added C58: 100nF, Capacitor_SMD:C_0603_1608Metric, B.Cu at (105.6, 55.6)
- added C59: 100nF, Capacitor_SMD:C_0603_1608Metric, B.Cu at (190.2, 58.6)
- added L1: 4.7uH, User_Footprints:L_TaiTech_HPC3010TF-4R7M, B.Cu at (101.5, 46.4)
- added U15: AP63205WU, Package_TO_SOT_SMD:TSOT-23-6, B.Cu at (97.6, 46.8)
- added U16: 74AHCT1G125, Package_TO_SOT_SMD:SOT-23-5, B.Cu at (159.2, 79.5)
- C16, C4: value 1nF -> 100nF
- C22, C23: value 1nF -> 10nF
- C31, C33, C35, C48, C50, C52: value 1nF -> 2.2nF
- R3, R30: value 120k -> 1M
- R33, R38, R58, R66: value 100k -> 180k
- R36, R64: value 100k -> 120k
- R37, R65: value 150k -> 270k
- R39, R67: value 33k -> 47k
- R4, R53: value 22k -> 470k
- U3: value AMS1117-5.0 -> AMS1117-3.3
- moved C6 72.2 mm to (114.9, 79.7)
- moved U3 66.7 mm to (167.7, 48.0)
- moved C4 58.6 mm to (183.8, 58.6), turned to 180 degrees
- moved C8 51.8 mm to (177.0, 61.3)
- moved C69 46.5 mm to (160.4, 89.1), turned to 0 degrees
- moved C16 19.9 mm to (127.8, 85.9), turned to 180 degrees
- moved C12 17.4 mm to (123.8, 68.9), turned to 0 degrees
- moved C42 12.4 mm to (107.7, 55.6)
- moved C7 3.64 mm to (169.5, 55.5)
- turned R3 to 90 degrees
- turned R30 to -90 degrees
- renumbered locked to SW2
Connections:
- C16 pad 1: Net-(C16-Pad1) -> +3.3VADC
- C16 pad 2: /sig_2 -> GND
- C4 pad 1: Net-(C4-Pad1) -> +3.3VADC
- C4 pad 2: /sig_1 -> GND
- C42 pad 1: +3V3 -> +3.3VADC
- C69 pad 1: +3V3 -> +3.3VADC
- R14 pad 2: Net-(C4-Pad1) -> Net-(U7A--)
- R15 pad 1: /trig_out_1 -> /Generator_Module1/trig_OUT
- R3 pad 1: REF-10 -> Net-(U7A--)
- R3 pad 2: Net-(C4-Pad1) -> REF-10
- R30 pad 1: REF-10 -> Net-(U7C--)
- R30 pad 2: Net-(C16-Pad1) -> REF-10
- R35 pad 2: Net-(C16-Pad1) -> Net-(U7C--)
- R4 pad 1: Net-(C4-Pad1) -> Net-(U7A--)
- R53 pad 1: Net-(C16-Pad1) -> Net-(U7C--)
- R72 pad 1: /trig_out_2 -> /Generator_Module2/trig_OUT
- RV12 pad 1: +3V3 -> +3.3VADC
- RV13 pad 1: +3V3 -> +3.3VADC
- RV4 pad 1: +3V3 -> +3.3VADC
- RV5 pad 1: +3V3 -> +3.3VADC
- SW2 pad : GND -> (no net)
- U10 pad 4: +3V3 -> +3.3VADC
- U11 pad 4: +3V3 -> +3.3VADC
- U13 pad 43: +3V3 -> +3.3VADC
- U3 pad 2: +5V -> +3.3VADC
- U3 pad 3: +12V -> +5V
- U7 pad 2: Net-(C4-Pad1) -> Net-(U7A--)
- U7 pad 4: +3V3 -> +3.3VADC
- U7 pad 9: Net-(C16-Pad1) -> Net-(U7C--)
Routing:
- net +3.3VADC: track 0.00 -> 330.2 mm, vias 0 -> 10
- net +3V3: track 409.1 -> 251.2 mm, vias 14 -> 11
- net Net-(U7C--): track 0.00 -> 96.5 mm, vias 0 -> 2
- net Net-(C16-Pad1): track 93.6 -> 0.00 mm, vias 2 -> 0
- net Net-(C4-Pad1): track 76.0 -> 0.00 mm
- net Net-(U7A--): track 0.00 -> 64.8 mm
- net GND: track 180.6 -> 209.9 mm, vias 29 -> 37
- net +5V: track 495.4 -> 509.3 mm
- net Net-(D18-DOUT): track 43.1 -> 35.9 mm
- net /LEDs/LED_data_in: track 6.45 -> 13.1 mm, vias 0 -> 2
- net Net-(U15-BST): track 0.00 -> 5.36 mm
- net /LED_data: track 9.02 -> 14.3 mm
- net Net-(Q2-Pad3): track 4.39 -> 0.00 mm
- net /lin_time_1: track 82.9 -> 79.9 mm
- net +12V: track 389.0 -> 391.4 mm, vias 10 -> 9
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Other:
- board text added: "BOOTSEL"
- board text added: "SPELLTWISTER v2.5"
- board text added: "have a good day!"
- board text removed: "SPELLTWISTER v2.0"

Commit message: beginning of pcb changes
Parts:
- added C3: 100nF, Capacitor_SMD:C_0603_1608Metric, F.Cu at (73.0, 77.0)
- added C60: 1uF, Capacitor_SMD:C_0603_1608Metric, F.Cu at (73.0, 79.5)
- added C61: 100nF, Capacitor_SMD:C_0603_1608Metric, F.Cu at (73.0, 82.0)
- added C62: 1uF, Capacitor_SMD:C_0603_1608Metric, F.Cu at (73.0, 84.5)
- C1, C2, C55, C56, C57, C7: value 10uF -> 22uF
- D10, D11, D12, D13, D14, D15, D16, D17, D18, D19, D20, D21, D22, D23, D24, D25, D3, D4, D5, D6, D7, D8, D9: footprint EURORACK:SK6812MINIE -> benjiaomodular:SK6812MINIE
- J10, J11, J12, J13, J14, J15, J16, J17, J18, J19, J2, J20, J4, J5, J6, J7, J8, J9: footprint EURORACK:AudioJack_3.5mm_with_drawing -> benjiaomodular:AudioJack_3.5mm_with_drawing
- RV1, RV10, RV14, RV2, RV3, RV6, RV7, RV8: footprint EURORACK:Potentiometer_RV09_talltrimmer -> benjiaomodular:Potentiometer_RV09_talltrimmer
- RV11, RV12, RV13, RV4, RV5, RV9: footprint EURORACK:Potentiometer_RV09_6mm_knob -> benjiaomodular:Potentiometer_RV09_6mm_knob
- SW1: footprint EURORACK:push_switch_5.1x5.1 -> benjiaomodular:push_switch_5.1x5.1
- SW2: footprint EURORACK:RotaryEncoder_Switch_Vertical_H20mm_20mm_knob -> benjiaomodular:RotaryEncoder_Switch_Vertical_H20mm_20mm_knob
- SW3: footprint EURORACK:SW_PUSH_6mm -> benjiaomodular:SW_PUSH_6mm
- SW4, SW5: footprint EURORACK:SPDT_P2.54mm_Vertical -> benjiaomodular:SPDT_P2.54mm_Vertical
- U16: footprint Package_TO_SOT_SMD:SOT-23-5 -> Package_TO_SOT_SMD:SOT-353_SC-70-5
- Y1: footprint EURORACK:ABM8-272-T3_ABR -> benjiaomodular:ABM8-272-T3_ABR
- moved L1 2.60 mm to (104.1, 46.4)
Connections:
- L1 pad 1: Net-(U15-BST) -> Net-(U15-SW)
- R15 pad 1: /Generator_Module1/trig_OUT -> /trig_out_1
- R72 pad 1: /Generator_Module2/trig_OUT -> /trig_out_2
- RV1 pad : GND -> (no net)
- RV10 pad : GND -> (no net)
- RV11 pad : GND -> (no net)
- RV12 pad : GND -> (no net)
- RV13 pad : GND -> (no net)
- RV14 pad : GND -> (no net)
- RV2 pad : GND -> (no net)
- RV3 pad : GND -> (no net)
- RV4 pad : GND -> (no net)
- RV5 pad : GND -> (no net)
- RV6 pad : GND -> (no net)
- RV7 pad : GND -> (no net)
- RV8 pad : GND -> (no net)
- RV9 pad : GND -> (no net)
Routing:
- net GND: track 209.9 -> 210.6 mm

Commit message: minor hardware changes
Parts:
- moved C1 39.3 mm to (184.5, 83.4)
- moved C57 12.5 mm to (202.8, 47.0), turned to 180 degrees
- moved C7 2.51 mm to (172.0, 55.5), turned to 180 degrees
- moved C2 2.29 mm to (91.8, 70.7), turned to 180 degrees
- moved C56 1.75 mm to (191.2, 54.2), turned to 180 degrees
Routing:
- net +3.3VADC: track 330.2 -> 345.4 mm
- net +12V: track 391.4 -> 397.1 mm
- net +3V3: track 251.2 -> 254.2 mm, vias 11 -> 10
- net /trig_out_2: track 6.58 -> 8.42 mm
- net +5V: track 509.7 -> 511.2 mm
- net -12V: track 192.3 -> 193.6 mm
Other:
- board text removed: "VCO LFO ENV"
- board text removed: "course pot"
- board text removed: "fine pot"
- board text removed: "follow btn"
- board text removed: "morph enc/btn"
- board text removed: "ratio att"
- board text removed: "ratio pot"
- board text removed: "shape att"
- board text removed: "shape pot"
- board text removed: "time att"
