File: hardware design/dsug_cctv_BOARD.kicad_sch (KiCad schematic)
At the start: 58 parts, among them J1 Conn_02x05_Top_Bottom, J3 TYPEC-304-ACP16, SW1 TS-1187A-B-A-B, SW2 24_detent, SW3 SW_Push, U1 AMS1117-3.3, U13 RP2040, U15 AP63205WU, U16 74AHCT1G125, U2 W25Q128JVS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

Commit message: library name updating, footprint swaps
Parts:
- SW1: footprint EURORACK:push_switch_5.1x5.1 -> benjiaomodular:push_switch_5.1x5.1
- SW2: footprint EURORACK:RotaryEncoder_Switch_Vertical_H20mm_20mm_knob -> benjiaomodular:RotaryEncoder_Switch_Vertical_H20mm_20mm_knob
- SW3: footprint EURORACK:SW_PUSH_6mm -> benjiaomodular:SW_PUSH_6mm
- U16: footprint Package_TO_SOT_SMD:SOT-23-5 -> Package_TO_SOT_SMD:SOT-353_SC-70-5
- Y1: footprint EURORACK:ABM8-272-T3_ABR -> benjiaomodular:ABM8-272-T3_ABR
Changed lines of the file:
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@@
 			)
 		)
-		(property "Footprint" "EURORACK:RotaryEncoder_Switch_Vertical_H20mm_20mm_knob"
+		(property "Footprint" "benjiaomodular:RotaryEncoder_Switch_Vertical_H20mm_20mm_knob"
 			(at 45.974 77.47 0)
 			(effects
@@
 			)
 		)
-		(property "Footprint" "EURORACK:push_switch_5.1x5.1"
+		(property "Footprint" "benjiaomodular:push_switch_5.1x5.1"
 			(at 204.978 55.372 0)
 			(effects
@@
 			)
 		)
-		(property "Footprint" "EURORACK:ABM8-272-T3_ABR"
+		(property "Footprint" "benjiaomodular:ABM8-272-T3_ABR"
 			(at 366.014 103.124 0)
 			(effects
@@
 			)
 		)
-		(property "Footprint" "EURORACK:SW_PUSH_6mm"
+		(property "Footprint" "benjiaomodular:SW_PUSH_6mm"
 			(at 41.91 115.316 0)
 			(effects
@@
 			)
 		)
-		(property "Footprint" "Package_TO_SOT_SMD:SOT-23-5"
+		(property "Footprint" "Package_TO_SOT_SMD:SOT-353_SC-70-5"
 			(at 67.31 35.56 0)
 			(effects

Commit message: minor hardware changes
Parts:
- added U17: 24LC01, symbol Memory_EEPROM:24LC01
Connections:
- net +3V3: now also U17.8 (VCC)
- net GND: now also U17.1 (A0), U17.2 (A1), U17.3 (A2), U17.4 (GND), U17.7 (WP)
